File: schematic/vumeter.sch (KiCad schematic (older format))
At the start: 9 parts

Commit message: updated a few values based on the final parts used
Parts:
- C12: value 0.1uF -> 0.47uF
- R18: value 1k_100k 1W -> 10k 1W
- RV2: value 1k_100K -> 47K
Changed lines of the file:
@@
 P 5800 3300
 F 0 "C12" H 5850 3500 50  0000 L CNN
-F 1 "0.1uF" H 5850 3400 50  0000 L CNN
+F 1 "0.47uF" H 5850 3400 50  0000 L CNN
 F 2 "Capacitor_THT:C_Axial_L22.0mm_D9.5mm_P27.50mm_Horizontal" H 5838 3150 50  0001 C CNN
 F 3 "~" H 5800 3300 50  0001 C CNN
@@
 P 7050 2950
 F 0 "R18" V 6843 2950 50  0000 C CNN
-F 1 "1k_100k 1W" V 6934 2950 50  0000 C CNN
+F 1 "10k 1W" V 6934 2950 50  0000 C CNN
 F 2 "Resistor_THT:R_Axial_DIN0411_L9.9mm_D3.6mm_P15.24mm_Horizontal" V 6980 2950 50  0001 C CNN
 F 3 "~" H 7050 2950 50  0001 C CNN
@@
 P 5400 2950
 F 0 "RV2" V 5193 2950 50  0000 C CNN
-F 1 "1k_100K" V 5284 2950 50  0000 C CNN
+F 1 "47K" V 5284 2950 50  0000 C CNN
 F 2 "Potentiometer_THT:Potentiometer_Piher_PT-6-V_Vertical" H 5400 2950 50  0001 C CNN
 F 3 "~" H 5400 2950 50  0001 C CNN
