File: schematic/power_regulator.sch (KiCad schematic (older format))
At the start: 15 parts, among them J1 Conn_01x02, Q1 TIP32A, Q2 2N3904, SW1 SW_SPST, T1 Transformer_1P_1S

Commit message: first decent version of dual channel opamp version.
Parts:
- D2: value 39 -> 39V
- F1: value 1A -> 2A
Changed lines of the file:
@@
 $Descr USLetter 11000 8500
 encoding utf-8
-Sheet 2 4
+Sheet 2 3
 Title "EL CHEAPO"
 Date "2021-01-05"
@@
 P 3500 3650
 F 0 "F1" V 3303 3650 50  0000 C CNN
-F 1 "1A" V 3394 3650 50  0000 C CNN
+F 1 "2A" V 3394 3650 50  0000 C CNN
 F 2 "" V 3430 3650 50  0001 C CNN
 F 3 "~" H 3500 3650 50  0001 C CNN
@@
 P 6900 4800
 F 0 "D2" V 6854 4879 50  0000 L CNN
-F 1 "39" V 6945 4879 50  0000 L CNN
+F 1 "39V" V 6945 4879 50  0000 L CNN
 F 2 "Diode_THT:D_DO-41_SOD81_P10.16mm_Horizontal" H 6900 4800 50  0001 C CNN
 F 3 "~" H 6900 4800 50  0001 C CNN
