File: schematic/el_cheapo.sch (KiCad schematic (older format))
At the start: 5 parts

Commit message: cleanup and remove resistor
Parts:
- removed H5: MountingHole_Pad, MountingHole:MountingHole_3.2mm_M3_Pad, symbol Mechanical:MountingHole_Pad
Connections:
- no-connect marks 1 -> 0
Changed lines of the file:
@@
 	5700 3950 5350 3950
-$Comp
-L Mechanical:MountingHole_Pad H5
-U 1 1 5FF6D28D
-P 8900 5700
-F 0 "H5" H 9000 5749 50  0000 L CNN
-F 1 "MountingHole_Pad" H 9000 5658 50  0000 L CNN
-F 2 "MountingHole:MountingHole_3.2mm_M3_Pad" H 8900 5700 50  0001 C CNN
-F 3 "~" H 8900 5700 50  0001 C CNN
-	1    8900 5700
-	1    0    0    -1
-$EndComp
 $Comp
 L Mechanical:MountingHole_Pad H4
@@
 	1    0    0    -1
 $EndComp
-NoConn ~ 8900 5800
 $EndSCHEMATC
